File: pcb/supermarketboard-left.kicad_pcb (KiCad board)
At the start: 2 copper layers, 180 x 130 mm, 84 parts, among them J1 PJ-320A-4P DIP

Commit message: asdflkadflkjahdfkjhafhjklasdffadsf
Parts:
- added LD1: SK6812MINI-E, LED_SMD:LED_SK6812MINI-E_3.2x2.8mm_P1.5mm_ReverseMount, B.Cu at (52.5, 44.0)
- added LD10: SK6812MINI-E, LED_SMD:LED_SK6812MINI-E_3.2x2.8mm_P1.5mm_ReverseMount, B.Cu at (138.0, 55.0)
- added LD11: SK6812MINI-E, LED_SMD:LED_SK6812MINI-E_3.2x2.8mm_P1.5mm_ReverseMount, B.Cu at (119.0, 60.5)
- added LD12: SK6812MINI-E, LED_SMD:LED_SK6812MINI-E_3.2x2.8mm_P1.5mm_ReverseMount, B.Cu at (100.0, 74.0)
- added LD13: SK6812MINI-E, LED_SMD:LED_SK6812MINI-E_3.2x2.8mm_P1.5mm_ReverseMount, B.Cu at (81.0, 74.0)
- added LD14: SK6812MINI-E, LED_SMD:LED_SK6812MINI-E_3.2x2.8mm_P1.5mm_ReverseMount, B.Cu at (62.0, 74.0)
- added LD15: SK6812MINI-E, LED_SMD:LED_SK6812MINI-E_3.2x2.8mm_P1.5mm_ReverseMount, B.Cu at (176.0, 82.0)
- added LD16: SK6812MINI-E, LED_SMD:LED_SK6812MINI-E_3.2x2.8mm_P1.5mm_ReverseMount, B.Cu at (157.0, 79.5)
- added LD17: SK6812MINI-E, LED_SMD:LED_SK6812MINI-E_3.2x2.8mm_P1.5mm_ReverseMount, B.Cu at (138.0, 74.0)
- added LD18: SK6812MINI-E, LED_SMD:LED_SK6812MINI-E_3.2x2.8mm_P1.5mm_ReverseMount, B.Cu at (119.0, 79.5)
- added LD19: SK6812MINI-E, LED_SMD:LED_SK6812MINI-E_3.2x2.8mm_P1.5mm_ReverseMount, B.Cu at (100.0, 93.0)
- added LD2: SK6812MINI-E, LED_SMD:LED_SK6812MINI-E_3.2x2.8mm_P1.5mm_ReverseMount, B.Cu at (81.0, 43.5)
- added LD20: SK6812MINI-E, LED_SMD:LED_SK6812MINI-E_3.2x2.8mm_P1.5mm_ReverseMount, B.Cu at (81.0, 93.0)
- added LD21: SK6812MINI-E, LED_SMD:LED_SK6812MINI-E_3.2x2.8mm_P1.5mm_ReverseMount, B.Cu at (57.2, 93.0)
- added LD22: SK6812MINI-E, LED_SMD:LED_SK6812MINI-E_3.2x2.8mm_P1.5mm_ReverseMount, B.Cu at (54.9, 112.0)
- added LD23: SK6812MINI-E, LED_SMD:LED_SK6812MINI-E_3.2x2.8mm_P1.5mm_ReverseMount, B.Cu at (81.0, 112.0)
- added LD24: SK6812MINI-E, LED_SMD:LED_SK6812MINI-E_3.2x2.8mm_P1.5mm_ReverseMount, B.Cu at (100.0, 112.0)
- added LD25: SK6812MINI-E, LED_SMD:LED_SK6812MINI-E_3.2x2.8mm_P1.5mm_ReverseMount, B.Cu at (119.0, 98.5)
- added LD26: SK6812MINI-E, LED_SMD:LED_SK6812MINI-E_3.2x2.8mm_P1.5mm_ReverseMount, B.Cu at (138.0, 93.0)
- added LD27: SK6812MINI-E, LED_SMD:LED_SK6812MINI-E_3.2x2.8mm_P1.5mm_ReverseMount, B.Cu at (157.0, 98.5)
- added LD28: SK6812MINI-E, LED_SMD:LED_SK6812MINI-E_3.2x2.8mm_P1.5mm_ReverseMount, B.Cu at (176.0, 101.0)
- added LD29: SK6812MINI-E, LED_SMD:LED_SK6812MINI-E_3.2x2.8mm_P1.5mm_ReverseMount, B.Cu at (52.5, 131.0)
- added LD3: SK6812MINI-E, LED_SMD:LED_SK6812MINI-E_3.2x2.8mm_P1.5mm_ReverseMount, B.Cu at (100.0, 44.0)
- added LD30: SK6812MINI-E, LED_SMD:LED_SK6812MINI-E_3.2x2.8mm_P1.5mm_ReverseMount, B.Cu at (81.0, 131.0)
- added LD31: SK6812MINI-E, LED_SMD:LED_SK6812MINI-E_3.2x2.8mm_P1.5mm_ReverseMount, B.Cu at (100.0, 131.0)
- added LD32: SK6812MINI-E, LED_SMD:LED_SK6812MINI-E_3.2x2.8mm_P1.5mm_ReverseMount, B.Cu at (119.0, 117.5)
- added LD33: SK6812MINI-E, LED_SMD:LED_SK6812MINI-E_3.2x2.8mm_P1.5mm_ReverseMount, B.Cu at (138.0, 112.0)
- added LD34: SK6812MINI-E, LED_SMD:LED_SK6812MINI-E_3.2x2.8mm_P1.5mm_ReverseMount, B.Cu at (157.0, 117.5)
- added LD35: SK6812MINI-E, LED_SMD:LED_SK6812MINI-E_3.2x2.8mm_P1.5mm_ReverseMount, B.Cu at (176.0, 120.0)
- added LD36: SK6812MINI-E, LED_SMD:LED_SK6812MINI-E_3.2x2.8mm_P1.5mm_ReverseMount, B.Cu at (195.0, 122.5)
- added LD37: SK6812MINI-E, LED_SMD:LED_SK6812MINI-E_3.2x2.8mm_P1.5mm_ReverseMount, B.Cu at (195.0, 145.5)
- added LD38: SK6812MINI-E, LED_SMD:LED_SK6812MINI-E_3.2x2.8mm_P1.5mm_ReverseMount, B.Cu at (176.0, 140.5)
- added LD39: SK6812MINI-E, LED_SMD:LED_SK6812MINI-E_3.2x2.8mm_P1.5mm_ReverseMount, B.Cu at (157.0, 136.5)
- added LD4: SK6812MINI-E, LED_SMD:LED_SK6812MINI-E_3.2x2.8mm_P1.5mm_ReverseMount, B.Cu at (119.0, 40.0)
- added LD40: SK6812MINI-E, LED_SMD:LED_SK6812MINI-E_3.2x2.8mm_P1.5mm_ReverseMount, B.Cu at (138.0, 131.0)
- added LD5: SK6812MINI-E, LED_SMD:LED_SK6812MINI-E_3.2x2.8mm_P1.5mm_ReverseMount, B.Cu at (138.0, 36.0)
- added LD6: SK6812MINI-E, LED_SMD:LED_SK6812MINI-E_3.2x2.8mm_P1.5mm_ReverseMount, B.Cu at (157.0, 40.0)
- added LD7: SK6812MINI-E, LED_SMD:LED_SK6812MINI-E_3.2x2.8mm_P1.5mm_ReverseMount, B.Cu at (176.0, 44.0)
- added LD8: SK6812MINI-E, LED_SMD:LED_SK6812MINI-E_3.2x2.8mm_P1.5mm_ReverseMount, B.Cu at (176.0, 63.0)
- added LD9: SK6812MINI-E, LED_SMD:LED_SK6812MINI-E_3.2x2.8mm_P1.5mm_ReverseMount, B.Cu at (157.0, 60.5)
- A1: moved to B.Cu
- moved A1 17.0 mm to (208.0, 38.5), turned to 180 degrees
Routing:
- net +3V3: track 0.00 -> 891.6 mm, vias 0 -> 52
- net COL1: track 0.00 -> 261.5 mm, vias 0 -> 1
- net COL3: track 0.00 -> 256.9 mm, vias 0 -> 1
- net COL4: track 0.00 -> 230.1 mm, vias 0 -> 2
- net COL2: track 0.00 -> 228.4 mm, vias 0 -> 1
- net COL5: track 0.00 -> 212.1 mm, vias 0 -> 1
- net ROW5: track 0.00 -> 208.2 mm, vias 0 -> 7
- net COL6: track 0.00 -> 193.0 mm, vias 0 -> 1
- net ROW1: track 0.00 -> 191.7 mm, vias 0 -> 8
- net ROW4: track 0.00 -> 186.1 mm, vias 0 -> 8
- net LED: track 0.00 -> 177.4 mm, vias 0 -> 2
- net ROW2: track 0.00 -> 175.4 mm, vias 0 -> 10
- net ROW3: track 0.00 -> 169.9 mm, vias 0 -> 8
- net COL7: track 0.00 -> 141.9 mm, vias 0 -> 1
- net ROW6: track 0.00 -> 125.1 mm, vias 0 -> 4
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- added copper zone on B.Cu, net GND
- added copper zone on F.Cu, net GND
Other:
- outline, holes or cut-outs redrawn
