File: pcb/supermarketboard-left.kicad_pcb (KiCad board)
At the start: 2 copper layers, 180 x 130 mm, 124 parts, among them J1 PJ-320A-4P DIP

Commit message: asdfhkjaksdfhjfasdjkhashkdfj
Parts:
- added H1: M3 Hole, MountingHole:MountingHole_3.2mm_M3_ISO7380_Pad, F.Cu at (90.5, 53.5)
- added H10: Bumpon, keys:Bumpon-Mirror, B.Cu at (187.5, 105.0)
- added H11: Bumpon, keys:Bumpon-Mirror, B.Cu at (69.0, 97.0)
- added H12: Bumpon, keys:Bumpon-Mirror, B.Cu at (127.3, 83.6)
- added H2: M3 Hole, MountingHole:MountingHole_3.2mm_M3_ISO7380_Pad, F.Cu at (90.5, 116.0)
- added H3: M3 Hole, MountingHole:MountingHole_3.2mm_M3_ISO7380_Pad, F.Cu at (165.5, 44.8)
- added H4: M3 Hole, MountingHole:MountingHole_3.2mm_M3_ISO7380_Pad, F.Cu at (167.5, 124.8)
- added H5: Bumpon, keys:Bumpon-Mirror, B.Cu at (62.0, 53.5)
- added H6: Bumpon, keys:Bumpon-Mirror, B.Cu at (40.0, 116.0)
- added H7: Bumpon, keys:Bumpon-Mirror, B.Cu at (127.0, 44.8)
- added H8: Bumpon, keys:Bumpon-Mirror, B.Cu at (127.0, 126.0)
- added H9: Bumpon, keys:Bumpon-Mirror, B.Cu at (184.9, 48.0)
- moved D37 3.80 mm to (165.5, 131.8)
Routing:
- net COL3: track 256.9 -> 262.0 mm
- net ROW6: track 125.1 -> 129.7 mm
- net Net-(D37-A): track 2.80 -> 6.13 mm
- net +3V3: track 891.6 -> 893.6 mm
- net COL6: track 193.0 -> 195.0 mm
- net LED: track 177.4 -> 178.6 mm
