File: pcb/supermarketboard-left.kicad_sch (KiCad schematic)
At the start: 4 parts, among them J1 PJ-320A-4P DIP

Commit message: asdflkadflkjahdfkjhafhjklasdffadsf
Other:
- added sheet LEDs (smbl-leds.kicad_sch)
Changed lines of the file:
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@@
+	)
+	(sheet
+		(at 139.7 165.1)
+		(size 12.7 3.81)
+		(exclude_from_sim no)
+		(in_bom yes)
+		(on_board yes)
+		(dnp no)
+		(fields_autoplaced yes)
+		(stroke
+			(width 0.1524)
+			(type solid)
+		)
+		(fill
+			(color 0 0 0 0)
+		)
+		(property "Sheetname" "LEDs"
+			(at 139.7 164.3884 0)
+			(show_name no)
+			(do_not_autoplace no)
+			(effects
+				(font
+					(size 1.27 1.27)
+				)
+				(justify left bottom)
+			)
+		)
+		(property "Sheetfile" "smbl-leds.kicad_sch"
+			(at 139.7 169.4946 0)
+			(show_name no)
+			(do_not_autoplace no)
+			(effects
+				(font
+					(size 1.27 1.27)
+				)
+				(justify left top)
+			)
+		)
+		(instances
+			(project "supermarketboard-left"
+				(path "/0dae0f32-c2d7-4dc8-95af-100ebdc818f4"
+					(page "3")
+				)
+			)
+		)
 	)
 	(sheet

Commit message: asdfhkjaksdfhjfasdjkhashkdfj
Parts:
- added H1, H2, H3, H4: M3 Hole, MountingHole:MountingHole_3.2mm_M3_ISO7380_Pad, symbol Mechanical:MountingHole_Pad
- added H10, H11, H12, H5, H6, H7, H8, H9: Bumpon, keys:Bumpon-Mirror, symbol Mechanical:MountingHole
Connections:
- net GND: now also H1.1, H2.1, H3.1, H4.1
